File: hardware/kicad/matrix_1.kicad_sch (KiCad schematic)
At the start: 155 parts, among them U5 IS31FL3741A

Commit message: update new led numbers
Parts:
- renumbered LED501 to LED410, LED502 to LED411, LED503 to LED412, LED504 to LED413, LED505 to LED414, LED506 to LED415, LED507 to LED416
Changed lines of the file:
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@@
 		(on_board yes)
 		(dnp no)
-		(property "Reference" "LED505"
+		(property "Reference" "LED414"
 			(at 201.295 238.125 0)
 			(effects
@@
 			(project "traffic_paradise"
 				(path "/911505fc-874d-4338-908e-12054bdd5112/11297df2-e2a9-48ca-8c4a-a4275dbea0eb"
-					(reference "LED505")
+					(reference "LED414")
 					(unit 1)
 				)
@@
 		(on_board yes)
 		(dnp no)
-		(property "Reference" "LED504"
+		(property "Reference" "LED413"
 			(at 188.595 238.125 0)
 			(effects
@@
 			(project "traffic_paradise"
 				(path "/911505fc-874d-4338-908e-12054bdd5112/11297df2-e2a9-48ca-8c4a-a4275dbea0eb"
-					(reference "LED504")
+					(reference "LED413")
 					(unit 1)
 				)
@@
 		(on_board yes)
 		(dnp no)
-		(property "Reference" "LED507"
+		(property "Reference" "LED416"
 			(at 252.095 200.025 0)
 			(effects
@@
 			(project "traffic_paradise"
 				(path "/911505fc-874d-4338-908e-12054bdd5112/11297df2-e2a9-48ca-8c4a-a4275dbea0eb"
-					(reference "LED507")
+					(reference "LED416")
 					(unit 1)
 				)
@@
 		(on_board yes)
 		(dnp no)
-		(property "Reference" "LED502"
+		(property "Reference" "LED411"
 			(at 163.195 238.125 0)
 			(effects
@@
 			(project "traffic_paradise"
 				(path "/911505fc-874d-4338-908e-12054bdd5112/11297df2-e2a9-48ca-8c4a-a4275dbea0eb"
-					(reference "LED502")
+					(reference "LED411")
 					(unit 1)
 				)
@@
 		(on_board yes)
 		(dnp no)
-		(property "Reference" "LED506"
+		(property "Reference" "LED415"
 			(at 213.995 238.125 0)
 			(effects
@@
 			(project "traffic_paradise"
 				(path "/911505fc-874d-4338-908e-12054bdd5112/11297df2-e2a9-48ca-8c4a-a4275dbea0eb"
-					(reference "LED506")
+					(reference "LED415")
 					(unit 1)
 				)
@@
 		(on_board yes)
 		(dnp no)
-		(property "Reference" "LED501"
+		(property "Reference" "LED410"
 			(at 150.495 238.125 0)
 			(effects
@@
 			(project "traffic_paradise"
 				(path "/911505fc-874d-4338-908e-12054bdd5112/11297df2-e2a9-48ca-8c4a-a4275dbea0eb"
-					(reference "LED501")
+					(reference "LED410")
 					(unit 1)
 				)
@@
 		(on_board yes)
 		(dnp no)
-		(property "Reference" "LED503"
+		(property "Reference" "LED412"
 			(at 175.895 238.125 0)
 			(effects
@@
 			(project "traffic_paradise"
 				(path "/911505fc-874d-4338-908e-12054bdd5112/11297df2-e2a9-48ca-8c4a-a4275dbea0eb"
-					(reference "LED503")
+					(reference "LED412")
 					(unit 1)
 				)

Commit message: fix small soldermask bridges and update production files
Parts:
- renumbered LED415 to LED325, LED410 to LED409, LED411 to LED410, LED412 to LED411, LED413 to LED412, LED414 to LED413, LED416 to LED414
Changed lines of the file:
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@@
 		(on_board yes)
 		(dnp no)
-		(property "Reference" "LED414"
+		(property "Reference" "LED413"
 			(at 201.295 238.125 0)
 			(effects
@@
 			(project "traffic_paradise"
 				(path "/911505fc-874d-4338-908e-12054bdd5112/11297df2-e2a9-48ca-8c4a-a4275dbea0eb"
-					(reference "LED414")
+					(reference "LED413")
 					(unit 1)
 				)
@@
 		(on_board yes)
 		(dnp no)
-		(property "Reference" "LED413"
+		(property "Reference" "LED412"
 			(at 188.595 238.125 0)
 			(effects
@@
 			(project "traffic_paradise"
 				(path "/911505fc-874d-4338-908e-12054bdd5112/11297df2-e2a9-48ca-8c4a-a4275dbea0eb"
-					(reference "LED413")
+					(reference "LED412")
 					(unit 1)
 				)
@@
 		(on_board yes)
 		(dnp no)
-		(property "Reference" "LED416"
+		(property "Reference" "LED414"
 			(at 252.095 200.025 0)
 			(effects
@@
 			(project "traffic_paradise"
 				(path "/911505fc-874d-4338-908e-12054bdd5112/11297df2-e2a9-48ca-8c4a-a4275dbea0eb"
-					(reference "LED416")
+					(reference "LED414")
 					(unit 1)
 				)
@@
 		(on_board yes)
 		(dnp no)
-		(property "Reference" "LED411"
+		(property "Reference" "LED410"
 			(at 163.195 238.125 0)
 			(effects
@@
 			(project "traffic_paradise"
 				(path "/911505fc-874d-4338-908e-12054bdd5112/11297df2-e2a9-48ca-8c4a-a4275dbea0eb"
-					(reference "LED411")
+					(reference "LED410")
 					(unit 1)
 				)
@@
 		(on_board yes)
 		(dnp no)
-		(property "Reference" "LED415"
+		(property "Reference" "LED325"
 			(at 213.995 238.125 0)
 			(effects
@@
 			(project "traffic_paradise"
 				(path "/911505fc-874d-4338-908e-12054bdd5112/11297df2-e2a9-48ca-8c4a-a4275dbea0eb"
-					(reference "LED415")
+					(reference "LED325")
 					(unit 1)
 				)
@@
 		(on_board yes)
 		(dnp no)
-		(property "Reference" "LED410"
+		(property "Reference" "LED409"
 			(at 150.495 238.125 0)
 			(effects
@@
 			(project "traffic_paradise"
 				(path "/911505fc-874d-4338-908e-12054bdd5112/11297df2-e2a9-48ca-8c4a-a4275dbea0eb"
-					(reference "LED410")
+					(reference "LED409")
 					(unit 1)
 				)
@@
 		(on_board yes)
 		(dnp no)
-		(property "Reference" "LED412"
+		(property "Reference" "LED411"
 			(at 175.895 238.125 0)
 			(effects
@@
 			(project "traffic_paradise"
 				(path "/911505fc-874d-4338-908e-12054bdd5112/11297df2-e2a9-48ca-8c4a-a4275dbea0eb"
-					(reference "LED412")
+					(reference "LED411")
 					(unit 1)
 				)
