File: hardware/kicad/matrix_4.kicad_sch (KiCad schematic)
At the start: 162 parts, among them U12 IS31FL3741A

Commit message: update new led numbers
Parts:
- renumbered LED401 to LED331, LED46 to LED332, LED335 to LED333, LED336 to LED334, LED337 to LED335, LED338 to LED336, LED339 to LED337, LED341 to LED338, LED342 to LED339, LED343 to LED340, LED344 to LED341, LED345 to LED342, LED346 to LED343, LED347 to LED344, LED348 to LED345, LED349 to LED346, LED350 to LED347, LED351 to LED348, LED352 to LED349, LED353 to LED350, LED354 to LED351, LED355 to LED352, LED356 to LED353, LED357 to LED354, LED358 to LED355, LED359 to LED356, LED360 to LED357, LED361 to LED358, LED402 to LED385, LED403 to LED386, LED404 to LED387, LED405 to LED388, LED406 to LED389, LED407 to LED390, LED408 to LED391, LED409 to LED392, LED410 to LED393, LED411 to LED394, LED412 to LED395, LED413 to LED396, LED414 to LED397, LED415 to LED398, LED416 to LED399, LED417 to LED400, LED418 to LED401, LED419 to LED402, LED420 to LED403, LED421 to LED404, LED422 to LED405, LED423 to LED406, LED424 to LED407, LED425 to LED408, LED426 to LED409

Commit message: fix small soldermask bridges and update production files
Parts:
- renumbered LED385 to LED384, LED386 to LED385, LED387 to LED386, LED388 to LED387, LED389 to LED388, LED390 to LED389, LED391 to LED390, LED392 to LED391, LED393 to LED392, LED394 to LED393, LED395 to LED394, LED396 to LED395, LED397 to LED396, LED398 to LED397, LED399 to LED398, LED400 to LED399, LED401 to LED400, LED402 to LED401, LED403 to LED402, LED404 to LED403, LED405 to LED404, LED406 to LED405, LED407 to LED406, LED408 to LED407, LED409 to LED408
Changed lines of the file:
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@@
 		(on_board yes)
 		(dnp no)
-		(property "Reference" "LED406"
+		(property "Reference" "LED405"
 			(at 188.595 257.175 0)
 			(effects
@@
 			(project "traffic_paradise"
 				(path "/911505fc-874d-4338-908e-12054bdd5112/229965e3-107a-47b9-9b24-fdc53810a62f"
-					(reference "LED406")
+					(reference "LED405")
 					(unit 1)
 				)
@@
 		(on_board yes)
 		(dnp no)
-		(property "Reference" "LED394"
+		(property "Reference" "LED393"
 			(at 150.495 238.125 0)
 			(effects
@@
 			(project "traffic_paradise"
 				(path "/911505fc-874d-4338-908e-12054bdd5112/229965e3-107a-47b9-9b24-fdc53810a62f"
-					(reference "LED394")
+					(reference "LED393")
 					(unit 1)
 				)
@@
 		(on_board yes)
 		(dnp no)
-		(property "Reference" "LED401"
+		(property "Reference" "LED400"
 			(at 239.395 238.125 0)
 			(effects
@@
 			(project "traffic_paradise"
 				(path "/911505fc-874d-4338-908e-12054bdd5112/229965e3-107a-47b9-9b24-fdc53810a62f"
-					(reference "LED401")
+					(reference "LED400")
 					(unit 1)
 				)
@@
 		(on_board yes)
 		(dnp no)
-		(property "Reference" "LED405"
+		(property "Reference" "LED404"
 			(at 175.895 257.175 0)
 			(effects
@@
 			(project "traffic_paradise"
 				(path "/911505fc-874d-4338-908e-12054bdd5112/229965e3-107a-47b9-9b24-fdc53810a62f"
-					(reference "LED405")
+					(reference "LED404")
 					(unit 1)
 				)
@@
 		(on_board yes)
 		(dnp no)
-		(property "Reference" "LED395"
+		(property "Reference" "LED394"
 			(at 163.195 238.125 0)
 			(effects
@@
 			(project "traffic_paradise"
 				(path "/911505fc-874d-4338-908e-12054bdd5112/229965e3-107a-47b9-9b24-fdc53810a62f"
-					(reference "LED395")
+					(reference "LED394")
 					(unit 1)
 				)
@@
 		(on_board yes)
 		(dnp no)
-		(property "Reference" "LED399"
+		(property "Reference" "LED398"
 			(at 213.995 238.125 0)
 			(effects
@@
 			(project "traffic_paradise"
 				(path "/911505fc-874d-4338-908e-12054bdd5112/229965e3-107a-47b9-9b24-fdc53810a62f"
-					(reference "LED399")
+					(reference "LED398")
 					(unit 1)
 				)
@@
 		(on_board yes)
 		(dnp no)
-		(property "Reference" "LED388"
+		(property "Reference" "LED387"
 			(at 188.595 219.075 0)
 			(effects
@@
 			(project "traffic_paradise"
 				(path "/911505fc-874d-4338-908e-12054bdd5112/229965e3-107a-47b9-9b24-fdc53810a62f"
-					(reference "LED388")
+					(reference "LED387")
 					(unit 1)
 				)
@@
 		(on_board yes)
 		(dnp no)
-		(property "Reference" "LED387"
+		(property "Reference" "LED386"
 			(at 175.895 219.075 0)
 			(effects
@@
 			(project "traffic_paradise"
 				(path "/911505fc-874d-4338-908e-12054bdd5112/229965e3-107a-47b9-9b24-fdc53810a62f"
-					(reference "LED387")
+					(reference "LED386")
 					(unit 1)
 				)
@@
 		(on_board yes)
 		(dnp no)
-		(property "Reference" "LED392"
+		(property "Reference" "LED391"
 			(at 239.395 219.075 0)
 			(effects
@@
 			(project "traffic_paradise"
 				(path "/911505fc-874d-4338-908e-12054bdd5112/229965e3-107a-47b9-9b24-fdc53810a62f"
-					(reference "LED392")
+					(reference "LED391")
 					(unit 1)
 				)
@@
 		(on_board yes)
 		(dnp no)
-		(property "Reference" "LED408"
+		(property "Reference" "LED407"
 			(at 213.995 257.175 0)
 			(effects
@@
 			(project "traffic_paradise"
 				(path "/911505fc-874d-4338-908e-12054bdd5112/229965e3-107a-47b9-9b24-fdc53810a62f"
-					(reference "LED408")
+					(reference "LED407")
 					(unit 1)
 				)
@@
 		(on_board yes)
 		(dnp no)
-		(property "Reference" "LED385"
+		(property "Reference" "LED384"
 			(at 150.495 219.075 0)
 			(effects
@@
 			(project "traffic_paradise"
 				(path "/911505fc-874d-4338-908e-12054bdd5112/229965e3-107a-47b9-9b24-fdc53810a62f"
-					(reference "LED385")
+					(reference "LED384")
 					(unit 1)
 				)
@@
 		(on_board yes)
 		(dnp no)
-		(property "Reference" "LED390"
+		(property "Reference" "LED389"
 			(at 213.995 219.075 0)
 			(effects
@@
 			(project "traffic_paradise"
 				(path "/911505fc-874d-4338-908e-12054bdd5112/229965e3-107a-47b9-9b24-fdc53810a62f"
-					(reference "LED390")
+					(reference "LED389")
 					(unit 1)
 				)
@@
 		(on_board yes)
 		(dnp no)
-		(property "Reference" "LED393"
+		(property "Reference" "LED392"
 			(at 252.095 219.075 0)
 			(effects
@@
 			(project "traffic_paradise"
 				(path "/911505fc-874d-4338-908e-12054bdd5112/229965e3-107a-47b9-9b24-fdc53810a62f"
-					(reference "LED393")
+					(reference "LED392")
 					(unit 1)
 				)
@@
 		(on_board yes)
 		(dnp no)
-		(property "Reference" "LED407"
+		(property "Reference" "LED406"
 			(at 201.295 257.175 0)
 			(effects
@@
 			(project "traffic_paradise"
 				(path "/911505fc-874d-4338-908e-12054bdd5112/229965e3-107a-47b9-9b24-fdc53810a62f"
-					(reference "LED407")
+					(reference "LED406")
 					(unit 1)
 				)
@@
 		(on_board yes)
 		(dnp no)
-		(property "Reference" "LED386"
+		(property "Reference" "LED385"
 			(at 163.195 219.075 0)
 			(effects
@@
 			(project "traffic_paradise"
 				(path "/911505fc-874d-4338-908e-12054bdd5112/229965e3-107a-47b9-9b24-fdc53810a62f"
-					(reference "LED386")
+					(reference "LED385")
 					(unit 1)
 				)
@@
 		(on_board yes)
 		(dnp no)
-		(property "Reference" "LED396"
+		(property "Reference" "LED395"
 			(at 175.895 238.125 0)
 			(effects
@@
 			(project "traffic_paradise"
 				(path "/911505fc-874d-4338-908e-12054bdd5112/229965e3-107a-47b9-9b24-fdc53810a62f"
-					(reference "LED396")
+					(reference "LED395")
 					(unit 1)
 				)
@@
 		(on_board yes)
 		(dnp no)
-		(property "Reference" "LED389"
+		(property "Reference" "LED388"
 			(at 201.295 219.075 0)
 			(effects
@@
 			(project "traffic_paradise"
 				(path "/911505fc-874d-4338-908e-12054bdd5112/229965e3-107a-47b9-9b24-fdc53810a62f"
-					(reference "LED389")
+					(reference "LED388")
 					(unit 1)
 				)
@@
 		(on_board yes)
 		(dnp no)
-		(property "Reference" "LED391"
+		(property "Reference" "LED390"
 			(at 226.695 219.075 0)
 			(effects
@@
 			(project "traffic_paradise"
 				(path "/911505fc-874d-4338-908e-12054bdd5112/229965e3-107a-47b9-9b24-fdc53810a62f"
-					(reference "LED391")
+					(reference "LED390")
 					(unit 1)
 				)
@@
 		(on_board yes)
 		(dnp no)
-		(property "Reference" "LED397"
+		(property "Reference" "LED396"
 			(at 188.595 238.125 0)
 			(effects
@@
 			(project "traffic_paradise"
 				(path "/911505fc-874d-4338-908e-12054bdd5112/229965e3-107a-47b9-9b24-fdc53810a62f"
-					(reference "LED397")
+					(reference "LED396")
 					(unit 1)
 				)
@@
 		(on_board yes)
 		(dnp no)
-		(property "Reference" "LED398"
+		(property "Reference" "LED397"
 			(at 201.295 238.125 0)
 			(effects
@@
 			(project "traffic_paradise"
 				(path "/911505fc-874d-4338-908e-12054bdd5112/229965e3-107a-47b9-9b24-fdc53810a62f"
-					(reference "LED398")
+					(reference "LED397")
 					(unit 1)
 				)
@@
 		(on_board yes)
 		(dnp no)
-		(property "Reference" "LED400"
+		(property "Reference" "LED399"
 			(at 226.695 238.125 0)
 			(effects
@@
 			(project "traffic_paradise"
 				(path "/911505fc-874d-4338-908e-12054bdd5112/229965e3-107a-47b9-9b24-fdc53810a62f"
-					(reference "LED400")
+					(reference "LED399")
 					(unit 1)
 				)
@@
 		(on_board yes)
 		(dnp no)
-		(property "Reference" "LED409"
+		(property "Reference" "LED408"
 			(at 226.695 257.175 0)
 			(effects
@@
 			(project "traffic_paradise"
 				(path "/911505fc-874d-4338-908e-12054bdd5112/229965e3-107a-47b9-9b24-fdc53810a62f"
-					(reference "LED409")
+					(reference "LED408")
 					(unit 1)
 				)
@@
 		(on_board yes)
 		(dnp no)
-		(property "Reference" "LED403"
+		(property "Reference" "LED402"
 			(at 150.495 257.175 0)
 			(effects
@@
 			(project "traffic_paradise"
 				(path "/911505fc-874d-4338-908e-12054bdd5112/229965e3-107a-47b9-9b24-fdc53810a62f"
-					(reference "LED403")
+					(reference "LED402")
 					(unit 1)
 				)
@@
 		(on_board yes)
 		(dnp no)
-		(property "Reference" "LED404"
+		(property "Reference" "LED403"
 			(at 163.195 257.175 0)
 			(effects
@@
 			(project "traffic_paradise"
 				(path "/911505fc-874d-4338-908e-12054bdd5112/229965e3-107a-47b9-9b24-fdc53810a62f"
-					(reference "LED404")
+					(reference "LED403")
 					(unit 1)
 				)
@@
 		(on_board yes)
 		(dnp no)
-		(property "Reference" "LED402"
+		(property "Reference" "LED401"
 			(at 252.095 238.125 0)
 			(effects
@@
 			(project "traffic_paradise"
 				(path "/911505fc-874d-4338-908e-12054bdd5112/229965e3-107a-47b9-9b24-fdc53810a62f"
-					(reference "LED402")
+					(reference "LED401")
 					(unit 1)
 				)
